Commit message: Add files via upload
Updated spawn function

File: urdf/pioneer3at_1.urdf (robot description, URDF)
Before this commit: robot pioneer3at, 17 links, 16 joints
Links:
- link base_link: mass 21.5 -> 31

File: urdf/pioneer3at_2.urdf (robot description, URDF)
Before this commit: robot pioneer3at, 17 links, 16 joints
Links:
- link base_link: mass 21.5 -> 31

File: urdf/pioneer3at_3.urdf (robot description, URDF)
Before this commit: robot pioneer3at, 17 links, 16 joints
Links:
- link base_link: mass 21.5 -> 31

File: urdf/pioneer3at_4.urdf (robot description, URDF)
Before this commit: robot pioneer3at, 17 links, 16 joints
Links:
- link base_link: mass 21.5 -> 31

File: urdf/pioneer3at_5.urdf (robot description, URDF)
Before this commit: robot pioneer3at, 17 links, 16 joints
Links:
- link base_link: mass 21.5 -> 31

Commit message: Add files via upload
Fixed spawn function

File: urdf/pioneer3at_1.urdf (robot description, URDF)
Before this commit: robot pioneer3at, 17 links, 16 joints
Links:
- added link hardener, mass 2; collision box size=0.05 0.05 0.01
- link base_link: mass 31 -> 26.5
Joints:
- added joint hardener_joint: type fixed, parent base_link, child hardener, origin xyz=0.16 0 0.074 rpy=0 0 0

File: urdf/pioneer3at_3.urdf (robot description, URDF)
Before this commit: robot pioneer3at, 17 links, 16 joints
Links:
- added link hardener, mass 2; collision box size=0.05 0.05 0.01
- link base_link: mass 31 -> 26.5
Joints:
- added joint hardener_joint: type fixed, parent base_link, child hardener, origin xyz=0.16 0 0.074 rpy=0 0 0

File: urdf/pioneer3at_4.urdf (robot description, URDF)
Before this commit: robot pioneer3at, 17 links, 16 joints
Links:
- added link hardener, mass 2; collision box size=0.05 0.05 0.01
- link base_link: mass 31 -> 26.5
Joints:
- added joint hardener_joint: type fixed, parent base_link, child hardener, origin xyz=0.16 0 0.074 rpy=0 0 0

File: urdf/pioneer3at_5.urdf (robot description, URDF)
Before this commit: robot pioneer3at, 17 links, 16 joints
Links:
- added link hardener, mass 2; collision box size=0.05 0.05 0.01
- link base_link: mass 31 -> 26.5
Joints:
- added joint hardener_joint: type fixed, parent base_link, child hardener, origin xyz=0.16 0 0.074 rpy=0 0 0

Commit message: Added weight for the target model to prevent rolls

File: urdf/pioneer3at_1.urdf (robot description, URDF)
Before this commit: robot pioneer3at, 18 links, 17 joints
Links:
- link hardener: mass 2 -> 4

File: urdf/pioneer3at_10.urdf (robot description, URDF)
Before this commit: robot pioneer3at, 18 links, 17 joints
Links:
- link hardener: mass 2 -> 4

File: urdf/pioneer3at_11.urdf (robot description, URDF)
Before this commit: robot pioneer3at, 18 links, 17 joints
Links:
- link hardener: mass 2 -> 4

File: urdf/pioneer3at_12.urdf (robot description, URDF)
Before this commit: robot pioneer3at, 18 links, 17 joints
Links:
- link hardener: mass 2 -> 4

File: urdf/pioneer3at_13.urdf (robot description, URDF)
Before this commit: robot pioneer3at, 18 links, 17 joints
Links:
- link hardener: mass 2 -> 4

File: urdf/pioneer3at_14.urdf (robot description, URDF)
Before this commit: robot pioneer3at, 18 links, 17 joints
Links:
- link hardener: mass 2 -> 4

File: urdf/pioneer3at_15.urdf (robot description, URDF)
Before this commit: robot pioneer3at, 18 links, 17 joints
Links:
- link hardener: mass 2 -> 4

File: urdf/pioneer3at_16.urdf (robot description, URDF)
Before this commit: robot pioneer3at, 18 links, 17 joints
Links:
- link hardener: mass 2 -> 4

File: urdf/pioneer3at_17.urdf (robot description, URDF)
Before this commit: robot pioneer3at, 18 links, 17 joints
Links:
- link hardener: mass 2 -> 4

File: urdf/pioneer3at_18.urdf (robot description, URDF)
Before this commit: robot pioneer3at, 18 links, 17 joints
Links:
- link hardener: mass 2 -> 4

File: urdf/pioneer3at_19.urdf (robot description, URDF)
Before this commit: robot pioneer3at, 18 links, 17 joints
Links:
- link hardener: mass 2 -> 4

File: urdf/pioneer3at_2.urdf (robot description, URDF)
Before this commit: robot pioneer3at, 18 links, 17 joints
Links:
- link hardener: mass 2 -> 4

File: urdf/pioneer3at_20.urdf (robot description, URDF)
Before this commit: robot pioneer3at, 18 links, 17 joints
Links:
- link hardener: mass 2 -> 4

File: urdf/pioneer3at_3.urdf (robot description, URDF)
Before this commit: robot pioneer3at, 18 links, 17 joints
Links:
- link hardener: mass 2 -> 4

File: urdf/pioneer3at_4.urdf (robot description, URDF)
Before this commit: robot pioneer3at, 18 links, 17 joints
Links:
- link hardener: mass 2 -> 4

File: urdf/pioneer3at_5.urdf (robot description, URDF)
Before this commit: robot pioneer3at, 18 links, 17 joints
Links:
- link hardener: mass 2 -> 4

File: urdf/pioneer3at_6.urdf (robot description, URDF)
Before this commit: robot pioneer3at, 18 links, 17 joints
Links:
- link hardener: mass 2 -> 4

File: urdf/pioneer3at_7.urdf (robot description, URDF)
Before this commit: robot pioneer3at, 18 links, 17 joints
Links:
- link hardener: mass 2 -> 4

File: urdf/pioneer3at_8.urdf (robot description, URDF)
Before this commit: robot pioneer3at, 18 links, 17 joints
Links:
- link hardener: mass 2 -> 4

File: urdf/pioneer3at_9.urdf (robot description, URDF)
Before this commit: robot pioneer3at, 18 links, 17 joints
Links:
- link hardener: mass 2 -> 4
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
Commit message: Added GPS plugin for targets

File: urdf/pioneer3at_1.urdf (robot description, URDF)
Before this commit: robot pioneer3at, 18 links, 17 joints
Joints:
- joint dir_point_joint: origin xyz=0.1 0 0 rpy=0 0 0 -> xyz=0.1 0 0.278 rpy=0 0 0

File: urdf/pioneer3at_2.urdf (robot description, URDF)
Before this commit: robot pioneer3at, 18 links, 17 joints
Joints:
- joint dir_point_joint: origin xyz=0.1 0 0 rpy=0 0 0 -> xyz=0.1 0 0.278 rpy=0 0 0
