Commit message: Logs added

File: urdf/pioneer3at_aruco.urdf (robot description, URDF)
Before this commit: robot pioneer3at, 19 links, 18 joints
Links:
- added link hardener, mass 4; collision box size=0.05 0.05 0.01
Joints:
- added joint hardener_joint: type fixed, parent base_link, child hardener, origin xyz=0.16 0 0.074 rpy=0 0 0

File: urdf/pioneer3at_cam.urdf (robot description, URDF)
Before this commit: robot pioneer3at, 18 links, 17 joints
Links:
- added link hardener, mass 4; collision box size=0.05 0.05 0.01
Joints:
- added joint hardener_joint: type fixed, parent base_link, child hardener, origin xyz=0.16 0 0.074 rpy=0 0 0
