Commit message: ORCA modified

File: urdf/hmap1/big_pioneer3at.urdf (robot description, URDF)
Before this commit: robot pioneer3at, 18 links, 17 joints
Links:
- link back_sonar: geometry visual mesh filename=package://amr_robots_description/meshes/p3at_meshes/back_so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 scale=2 2 2
- link base_link: geometry collision mesh filename=package://amr_robots_description/meshes/p3at_meshes/chassis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 scale=2 2 2; visual mesh filename=package://amr_robots_description/meshes/p3at_meshes/chassis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 scale=2 2 2
- link front_sonar: geometry visual mesh filename=package://amr_robots_description/meshes/p3at_meshes/front_s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 scale=2 2 2
- link p3at_back_left_axle: geometry collision mesh filename=package://amr_robots_description/meshes/p3at_meshes/axle.stl scale=2 2 2; visual mesh filename=package://amr_robots_description/meshes/p3at_meshes/axle.stl scale=2 2 2
- link p3at_back_left_hub: geometry collision mesh filename=package://amr_robots_description/meshes/p3at_meshes/left_hu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 scale=2 2 2; visual mesh filename=package://amr_robots_description/meshes/p3at_meshes/left_hu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 scale=2 2 2
- link p3at_back_left_wheel: geometry collision cylinder length=0.075 radius=0.111; visual mesh filename=package://amr_robots_description/meshes/p3at_meshes/wheel.s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 scale=2 2 2
- link p3at_back_right_axle: geometry collision mesh filename=package://amr_robots_description/meshes/p3at_meshes/axle.stl scale=2 2 2; visual mesh filename=package://amr_robots_description/meshes/p3at_meshes/axle.stl scale=2 2 2
- link p3at_back_right_hub: geometry collision mesh filename=package://amr_robots_description/meshes/p3at_meshes/right_h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 scale=2 2 2; visual mesh filename=package://amr_robots_description/meshes/p3at_meshes/right_h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 scale=2 2 2
- link p3at_back_right_wheel: geometry collision cylinder length=0.075 radius=0.111; visual mesh filename=package://amr_robots_description/meshes/p3at_meshes/wheel.s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 scale=2 2 2
- link p3at_front_left_axle: geometry visual mesh filename=package://amr_robots_description/meshes/p3at_meshes/axle.stl scale=2 2 2
- link p3at_front_left_hub: geometry visual mesh filename=package://amr_robots_description/meshes/p3at_meshes/left_hu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 scale=2 2 2
- link p3at_front_left_wheel: geometry collision cylinder length=0.075 radius=0.111; visual mesh filename=package://amr_robots_description/meshes/p3at_meshes/wheel.s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 scale=2 2 2
- link p3at_front_right_axle: geometry visual mesh filename=package://amr_robots_description/meshes/p3at_meshes/axle.stl scale=2 2 2
- link p3at_front_right_hub: geometry visual mesh filename=package://amr_robots_description/meshes/p3at_meshes/right_h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 scale=2 2 2
- link p3at_front_right_wheel: geometry collision cylinder length=0.075 radius=0.111; visual mesh filename=package://amr_robots_description/meshes/p3at_meshes/wheel.s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 scale=2 2 2
- link top_plate: geometry visual mesh filename=package://amr_robots_description/meshes/p3at_meshes/top.stl scale=2 2 2

Commit message: ORCA modified

File: urdf/hmap1/big_pioneer3at.urdf (robot description, URDF)
Before this commit: robot pioneer3at, 18 links, 17 joints
Links:
- added link world
- link back_sonar: geometry visual mesh filename=package://amr_robots_description/meshes/p3at_meshes/back_so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 scale=4 4 4
- link base_link: mass 26.5 -> 344; geometry collision mesh filename=package://amr_robots_description/meshes/p3at_meshes/chassis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 scale=4 4 4; visual mesh filename=package://amr_robots_description/meshes/p3at_meshes/chassis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 scale=4 4 4
- link dir_point: geometry visual sphere radius=0.04
- link front_sonar: geometry visual mesh filename=package://amr_robots_description/meshes/p3at_meshes/front_s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 scale=4 4 4
- link hardener: geometry collision box size=0.2 0.2 0.04
- link p3at_back_left_axle: geometry collision mesh filename=package://amr_robots_description/meshes/p3at_meshes/axle.stl scale=4 4 4; visual mesh filename=package://amr_robots_description/meshes/p3at_meshes/axle.stl scale=4 4 4
- link p3at_back_left_hub: geometry collision mesh filename=package://amr_robots_description/meshes/p3at_meshes/left_hu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 scale=4 4 4; visual mesh filename=package://amr_robots_description/meshes/p3at_meshes/left_hu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 scale=4 4 4
- link p3at_back_left_wheel: mass 1.2 -> 19.2; geometry collision cylinder length=0.3 radius=0.444; visual mesh filename=package://amr_robots_description/meshes/p3at_meshes/wheel.s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 scale=4 4 4
- link p3at_back_right_axle: geometry collision mesh filename=package://amr_robots_description/meshes/p3at_meshes/axle.stl scale=4 4 4; visual mesh filename=package://amr_robots_description/meshes/p3at_meshes/axle.stl scale=4 4 4
- link p3at_back_right_hub: geometry collision mesh filename=package://amr_robots_description/meshes/p3at_meshes/right_h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 scale=4 4 4; visual mesh filename=package://amr_robots_description/meshes/p3at_meshes/right_h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 scale=4 4 4
- link p3at_back_right_wheel: mass 1.2 -> 19.2; geometry collision cylinder length=0.3 radius=0.444; visual mesh filename=package://amr_robots_description/meshes/p3at_meshes/wheel.s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 scale=4 4 4
- link p3at_front_left_axle: geometry visual mesh filename=package://amr_robots_description/meshes/p3at_meshes/axle.stl scale=4 4 4
- link p3at_front_left_hub: geometry visual mesh filename=package://amr_robots_description/meshes/p3at_meshes/left_hu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 scale=4 4 4
- link p3at_front_left_wheel: mass 1.2 -> 19.2; geometry collision cylinder length=0.3 radius=0.444; visual mesh filename=package://amr_robots_description/meshes/p3at_meshes/wheel.s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 scale=4 4 4
- link p3at_front_right_axle: geometry visual mesh filename=package://amr_robots_description/meshes/p3at_meshes/axle.stl scale=4 4 4
- link p3at_front_right_hub: geometry visual mesh filename=package://amr_robots_description/meshes/p3at_meshes/right_h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 scale=4 4 4
- link p3at_front_right_wheel: mass 1.2 -> 19.2; geometry collision cylinder length=0.3 radius=0.444; visual mesh filename=package://amr_robots_description/meshes/p3at_meshes/wheel.s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 scale=4 4 4
- link top_plate: geometry visual mesh filename=package://amr_robots_description/meshes/p3at_meshes/top.stl scale=4 4 4
Joints:
- added joint fixed: type fixed, parent world, child base_link
- joint base_back_joint: origin xyz=-0.187 0 0.247 rpy=0 0 0 -> xyz=-0.748 0 0.988 rpy=0 0 0
- joint base_front_joint: origin xyz=0.193 0 0.25 rpy=0 0 0 -> xyz=0.772 0 1 rpy=0 0 0
- joint base_front_left_axle_joint: origin xyz=0.135 0.156 0.111 rpy=0 0 0 -> xyz=0.540 0.624 0.444 rpy=0 0 0
- joint base_front_left_hub_joint: origin xyz=0 0.041 0 rpy=0 0 0 -> xyz=0 0.164 0 rpy=0 0 0
- joint base_front_right_axle_joint: origin xyz=0.135 -0.156 0.111 rpy=0 0 0 -> xyz=0.540 -0.624 0.444 rpy=0 0 0
- joint base_front_right_hub_joint: origin xyz=0 -0.041 0 rpy=0 0 0 -> xyz=0 -0.164 0 rpy=0 0 0
- joint base_top_joint: origin xyz=0.003 0 0.274 rpy=0 0 0 -> xyz=0.012 0 1.096 rpy=0 0 0
- joint dir_point_joint: origin xyz=0.1 0 0.278 rpy=0 0 0 -> xyz=0.1 0 1.112 rpy=0 0 0
- joint hardener_joint: origin xyz=0.16 0 0.074 rpy=0 0 0 -> xyz=0.64 0 0.296 rpy=0 0 0
- joint p3at_back_left_axle_joint: origin xyz=-0.134 0.156 0.111 rpy=0 0 0 -> xyz=-0.540 0.624 0.444 rpy=0 0 0
- joint p3at_back_left_hub_joint: origin xyz=-0 0.041 0 rpy=0 0 0 -> xyz=-0 0.164 0 rpy=0 0 0
- joint p3at_back_right_axle_joint: origin xyz=-0.134 -0.156 0.111 rpy=0 0 0 -> xyz=-0.540 -0.624 0.444 rpy=0 0 0
- joint p3at_back_right_hub_joint: origin xyz=-0 -0.041 0 rpy=0 0 0 -> xyz=-0 -0.164 0 rpy=0 0 0
