Commit message: New paths added

File: urdf/hmap2/big_pioneer3at.urdf (robot description, URDF)
Before this commit: robot pioneer3at, 18 links, 17 joints
Links:
- removed link back_sonar
- removed link front_sonar
- removed link hardener
- link base_link: mass 26.5 -> 344; geometry collision box size=1.25 1 0.7; visual mesh filename=package://amr_robots_description/meshes/p3at_meshes/chassis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 scale=4 4 4
- link dir_point: geometry visual sphere radius=0.04
- link p3at_back_left_axle: geometry visual mesh filename=package://amr_robots_description/meshes/p3at_meshes/axle.stl scale=4 4 4
- link p3at_back_left_hub: geometry visual mesh filename=package://amr_robots_description/meshes/p3at_meshes/left_hu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 scale=4 4 4
- link p3at_back_left_wheel: mass 1.2 -> 19.2; geometry collision cylinder length=0.3 radius=0.444; visual mesh filename=package://amr_robots_description/meshes/p3at_meshes/wheel.s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 scale=4 4 4
- link p3at_back_right_axle: geometry visual mesh filename=package://amr_robots_description/meshes/p3at_meshes/axle.stl scale=4 4 4
- link p3at_back_right_hub: geometry visual mesh filename=package://amr_robots_description/meshes/p3at_meshes/right_h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 scale=4 4 4
- link p3at_back_right_wheel: mass 1.2 -> 19.2; geometry collision cylinder length=0.3 radius=0.444; visual mesh filename=package://amr_robots_description/meshes/p3at_meshes/wheel.s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 scale=4 4 4
- link p3at_front_left_axle: geometry visual mesh filename=package://amr_robots_description/meshes/p3at_meshes/axle.stl scale=4 4 4
- link p3at_front_left_hub: geometry visual mesh filename=package://amr_robots_description/meshes/p3at_meshes/left_hu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 scale=4 4 4
- link p3at_front_left_wheel: mass 1.2 -> 19.2; geometry collision cylinder length=0.3 radius=0.444; visual mesh filename=package://amr_robots_description/meshes/p3at_meshes/wheel.s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 scale=4 4 4
- link p3at_front_right_axle: geometry visual mesh filename=package://amr_robots_description/meshes/p3at_meshes/axle.stl scale=4 4 4
- link p3at_front_right_hub: geometry visual mesh filename=package://amr_robots_description/meshes/p3at_meshes/right_h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 scale=4 4 4
- link p3at_front_right_wheel: mass 1.2 -> 19.2; geometry collision cylinder length=0.3 radius=0.444; visual mesh filename=package://amr_robots_description/meshes/p3at_meshes/wheel.s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 scale=4 4 4
- link top_plate: geometry visual mesh filename=package://amr_robots_description/meshes/p3at_meshes/top.stl scale=4 4 4
Joints:
- removed joint base_back_joint
- removed joint base_front_joint
- removed joint hardener_joint
- joint base_front_left_axle_joint: origin xyz=0.135 0.156 0.111 rpy=0 0 0 -> xyz=0.540 0.624 0.444 rpy=0 0 0
- joint base_front_left_hub_joint: origin xyz=0 0.041 0 rpy=0 0 0 -> xyz=0 0.164 0 rpy=0 0 0
- joint base_front_right_axle_joint: origin xyz=0.135 -0.156 0.111 rpy=0 0 0 -> xyz=0.540 -0.624 0.444 rpy=0 0 0
- joint base_front_right_hub_joint: origin xyz=0 -0.041 0 rpy=0 0 0 -> xyz=0 -0.164 0 rpy=0 0 0
- joint base_top_joint: origin xyz=0.003 0 0.274 rpy=0 0 0 -> xyz=0.012 0 1.096 rpy=0 0 0
- joint dir_point_joint: origin xyz=0.1 0 0.278 rpy=0 0 0 -> xyz=0.1 0 1.112 rpy=0 0 0
- joint p3at_back_left_axle_joint: origin xyz=-0.134 0.156 0.111 rpy=0 0 0 -> xyz=-0.536 0.624 0.444 rpy=0 0 0
- joint p3at_back_left_hub_joint: origin xyz=-0 0.041 0 rpy=0 0 0 -> xyz=-0 0.164 0 rpy=0 0 0
- joint p3at_back_right_axle_joint: origin xyz=-0.134 -0.156 0.111 rpy=0 0 0 -> xyz=-0.536 -0.624 0.444 rpy=0 0 0
- joint p3at_back_right_hub_joint: origin xyz=-0 -0.041 0 rpy=0 0 0 -> xyz=-0 -0.164 0 rpy=0 0 0
