Commit message: Big targets deleted

File: urdf/hmap2/pioneer3at.urdf (robot description, URDF)
Before this commit: robot pioneer3at, 18 links, 17 joints
Links:
- removed link hardener
Joints:
- removed joint hardener_joint

Commit message: Target model fixed

File: urdf/hmap2/pioneer3at.urdf (robot description, URDF)
Before this commit: robot pioneer3at, 17 links, 16 joints
Links:
- added link hardener, mass 4; collision box size=0.05 0.05 0.01
Joints:
- added joint hardener_joint: type fixed, parent base_link, child hardener, origin xyz=0.16 0 0.074 rpy=0 0 0
